Commit message: publish speed and convert vel of wheels

File: src/mybot_description/urdf/mybot.xacro (robot description, xacro)
@@ -6,4 +6,5 @@
   <xacro:include filename="$(find mybot_description)/urdf/materials.xacro" />
   <xacro:include filename="$(find mybot_description)/urdf/macros.xacro" />
+  <link name = "base_link" />
   <link name='chassis'>
     <pose>0 0 0.1 0 0 0</pose>
